File: kicad_projects/typeS/Phoenix_Project_No1-TypeS.kicad_sch (KiCad schematic)
At the start: 66 parts, among them J1 USB_B_Mini, J2 SWD, J3 Shield, SW1 K2-1187SQ-A4SW-06, SW2 K2-1187SQ-A4SW-06, U1 ADP122AUJZ-3.3-R7, U2 TPD3E001DRLR, U3 RP2040, U4 W25Q16JVUXIQ, Y1 12MHz

Commit message: [feature] New Type S PCB Rev 2.1
This fixes wrong placement of split backspace keys.
Parts:
- H1, H2: footprint mymakercorner:The_Phoenix_Project_No1_TypeS_Rev2_Logo -> mymakercorner:The_Phoenix_Project_No1_TypeS_Rev2_1_Logo
Changed lines of the file:
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@@
   (title_block
     (title "Phoenix Project No 1 - Type S")
-    (date "2023-05-07")
-    (rev "2")
+    (date "2024-07-13")
+    (rev "2.1")
     (comment 1 "Designed with love by Rico")
   )
@@
       (effects (font (size 1.27 1.27)) (justify left))
     )
-    (property "Footprint" "mymakercorner:The_Phoenix_Project_No1_TypeS_Rev2_Logo" (id 2) (at 200.025 268.605 0)
+    (property "Footprint" "mymakercorner:The_Phoenix_Project_No1_TypeS_Rev2_1_Logo" (id 2) (at 200.025 268.605 0)
       (effects (font (size 1.27 1.27)) hide)
     )
@@
       (effects (font (size 1.27 1.27)) (justify left))
     )
-    (property "Footprint" "mymakercorner:The_Phoenix_Project_No1_TypeS_Rev2_Logo" (id 2) (at 200.025 262.255 0)
+    (property "Footprint" "mymakercorner:The_Phoenix_Project_No1_TypeS_Rev2_1_Logo" (id 2) (at 200.025 262.255 0)
       (effects (font (size 1.27 1.27)) hide)
     )
@@
     )
     (path "/77e9c9e6-4e9a-435e-b8b5-389d514213e0"
-      (reference "H1") (unit 1) (value "Phoenix_Projet_TypeS_Rev2_Front") (footprint "mymakercorner:The_Phoenix_Project_No1_TypeS_Rev2_Logo")
+      (reference "H1") (unit 1) (value "Phoenix_Projet_TypeS_Rev2_Front") (footprint "mymakercorner:The_Phoenix_Project_No1_TypeS_Rev2_1_Logo")
     )
     (path "/74665f50-fc4e-4807-bd95-689e28b8585c"
-      (reference "H2") (unit 1) (value "Phoenix_Projet_TypeS_Rev2_Back") (footprint "mymakercorner:The_Phoenix_Project_No1_TypeS_Rev2_Logo")
+      (reference "H2") (unit 1) (value "Phoenix_Projet_TypeS_Rev2_Back") (footprint "mymakercorner:The_Phoenix_Project_No1_TypeS_Rev2_1_Logo")
     )
     (path "/5fa9667e-006a-4108-aa96-ff067b1783a5"
